Commit message: add arcl_youbot_application

File: luh_youbot_description/urdf/youbot_base/base.urdf.xacro (robot description, xacro)
@@ -13,5 +13,8 @@
       <property name="wheel_offset_y" value="0.158"  />
       <property name="wheel_offset_z" value="-0.034" />
-    <property name="wheel_mass" value="0.4" />
+    <!-- <property name="wheel_mass" value="0.4" /> -->
+    <!-- DEBUG-->
+    <property name="wheel_mass" value="4" />
+    <!--END DEBUG-->
     <property name="wheel_radius" value="0.05" />
     <property name="wheel_length" value="0.07" />

File: luh_youbot_description/urdf/youbot_plate/plate.urdf.xacro (robot description, xacro)
@@ -11,5 +11,5 @@
 			<inertial>
 				<origin xyz="0 0 0" rpy="0 0 0"/>
-				<mass value="1"/>
+				<mass value="10"/>
 				<inertia ixx="0.001" ixy="0" ixz="0" iyy="0.001" iyz="0" izz="0.001" />
 			</inertial>
