Commit message: grasp plugin

File: luh_youbot_description/robots/youbot_gazebo.xacro (robot description, xacro)
@@ -10,3 +10,29 @@
      </gazebo>
   </xacro:macro>
+  <xacro:macro name="gzplugin_grasp_fix">
+	<gazebo>
+		<plugin name="gazebo_grasp_fix" filename="libgazebo_grasp_fix.so">
+			<!--
+            NOTE: The finger tips are linked together with the links before, because they are connected with a
+			fixed joint. Gazebo makes one whole link out of this automatically. When listing the 9_*_tip links
+			here, they won't be found in the SDF.
+<max_grip_count>8</max_grip_count>
+            <release_tolerance>0.007</release_tolerance>
+            -->
+            <arm>
+                <arm_name>youbot</arm_name>
+                <palm_link>arm_link_5</palm_link>
+                <gripper_link>gripper_finger_link_r</gripper_link>
+                <gripper_link>gripper_finger_link_l</gripper_link>
+            </arm>
+            <forces_angle_tolerance>100</forces_angle_tolerance>
+            <update_rate>4</update_rate>
+            <grip_count_threshold>1</grip_count_threshold>
+            <max_grip_count>8</max_grip_count>
+            <release_tolerance>0.007</release_tolerance>
+            <disable_collisions_on_attach>false</disable_collisions_on_attach>
+            <contact_topic>__default_topic__</contact_topic>
+		</plugin>
+	</gazebo>
+</xacro:macro>
 </robot>
