Commit message: change gripper

File: luh_youbot_description/robots/youbot.urdf.xacro (robot description, xacro)
@@ -27,8 +27,8 @@
   </xacro:youbot_gripper>
   <!-- Kamera -->
-  <xacro:include filename="$(find luh_youbot_description)/urdf/sensors/asus_xtion_camera.urdf.xacro" />
+  <!-- <xacro:include filename="$(find luh_youbot_description)/urdf/sensors/asus_xtion_camera.urdf.xacro" />
   <xacro:asus_xtion_camera name="camera" parent="arm_link_5" tilt="0.0">
     <origin xyz="-0.02 0 -0.04" rpy="0 -1.60 0" />
-  </xacro:asus_xtion_camera>
+  </xacro:asus_xtion_camera> -->
   <xacro:joint_state_publisher namespace="gazebo"/>
 </robot>

File: luh_youbot_description/urdf/sensors/hokuyo_urg04_laser.urdf.xacro (robot description, xacro)
@@ -24,5 +24,5 @@
 		<origin xyz="0 0 0" rpy="0 0 0" />
 		<geometry>
-			<mesh filename="package://luh_youbot_description/meshes/sensors/hokuyo_convex.dae" />
+			<!-- <mesh filename="package://luh_youbot_description/meshes/sensors/hokuyo_convex.dae" />			 -->
 		</geometry>
 	</collision>

File: luh_youbot_description/urdf/youbot_base/base.urdf.xacro (robot description, xacro)
@@ -2,7 +2,7 @@
 <robot  xmlns:xacro="http://ros.org/wiki/xacro">
     <!-- sensors -->
-    <xacro:include filename="$(find luh_youbot_description)/urdf/sensors/hokuyo_urg04_laser.urdf.xacro"/>
+    <!-- <xacro:include filename="$(find luh_youbot_description)/urdf/sensors/hokuyo_urg04_laser.urdf.xacro"/> -->
   <xacro:include filename="$(find luh_youbot_description)/urdf/youbot_base/base.gazebo.xacro" />
-  <xacro:include filename="$(find luh_youbot_description)/urdf/youbot_base/bumper.gazebo.xacro" />
+  <!-- <xacro:include filename="$(find luh_youbot_description)/urdf/youbot_base/bumper.gazebo.xacro" /> -->
      <!-- simplified box collision geometry for base -->
       <property name="base_size_x" value="0.570" />
@@ -62,16 +62,17 @@
                     <origin xyz="0 0 0" rpy="0 0 0" />
                     <geometry>
-                    <mesh filename="package://luh_youbot_description/meshes/youbot_base/base_convex.dae"/>
+                    <mesh filename="package://luh_youbot_description/meshes/youbot_base/base_convex_small.dae"/>
                        </geometry>
                   </collision>
             </link>
         <!-- base laser front -->
-            <xacro:hokuyo_urg04_laser name="${name}_laser_front" parent="${name}" ros_topic="scan" update_rate="10" min_angle="-1.57" max_angle="1.57" >
+            <!-- <xacro:hokuyo_urg04_laser name="${name}_laser_front" parent="${name}" ros_topic="scan" update_rate="10" min_angle="-1.57" max_angle="1.57" >
                   <origin xyz="0.309 0 -0.03" rpy="0 0 0" />
-            </xacro:hokuyo_urg04_laser>
+            </xacro:hokuyo_urg04_laser> -->
         <!-- base laser back -->
-            <xacro:hokuyo_urg04_laser  name="${name}_laser_back" parent="${name}" ros_topic="scan_back" update_rate="10" min_angle="1.57" max_angle="-1.57" >
+            <!-- <xacro:hokuyo_urg04_laser  name="${name}_laser_back" parent="${name}" ros_topic="scan_back" update_rate="10" min_angle="1.57" max_angle="-1.57" >
                   <origin xyz="-0.309 0 -0.03" rpy="0 0 ${M_PI}" />
             </xacro:hokuyo_urg04_laser>
+         -->
             <!-- front left wheel -->
         <joint name="wheel_joint_fl" type="continuous">
@@ -195,5 +196,5 @@
             </link>
         <xacro:youbot_base_controller namespace="gazebo"/>
-        <xacro:youbot_base_bumper namespace="${namespace}"/>
+        <!-- <xacro:youbot_base_bumper namespace="${namespace}"/> -->
     </xacro:macro>
 </robot>

File: luh_youbot_description/urdf/youbot_gripper/gripper.urdf.xacro (robot description, xacro)
@@ -1,102 +1,113 @@
 <?xml version="1.0"?>
 <robot xmlns:xacro="http://ros.org/wiki/xacro">
-    <xacro:include filename="$(find luh_youbot_description)/urdf/youbot_gripper/limits.urdf.xacro" />
-    <xacro:include filename="$(find luh_youbot_description)/urdf/youbot_gripper/gripper.gazebo.xacro" />
-    <xacro:macro name="youbot_gripper" params="parent name namespace *origin">
-        <!-- joint between arm_7_link and sdh_palm_link -->
-        <joint name="${name}_palm_joint" type="fixed" >
-            <insert_block name="origin" />
-            <parent link="${parent}" />
-            <child link="${name}_palm_link" />
-        </joint>
-        <link name="${name}_palm_link">
-            <inertial>
-                <origin xyz="0 0 0" rpy="0 0 0"/>
-                <mass value="0.1"/>
-                <inertia ixx="0.0001" ixy="0" ixz="0" iyy="0.0001" iyz="0" izz="0.0001" />
-            </inertial>
-            <visual>
-                <origin xyz="0 0 -0.0139" rpy="0 ${-M_PI/2} ${M_PI/2}"/>
-                <geometry>
-                    <mesh filename="package://luh_youbot_description/meshes/youbot_gripper/palm.dae" />
-                </geometry>
-            </visual>
-            <collision>
-                <origin xyz="0.003 0 0.01" rpy="0 0 0" />
-                <geometry>
-                    <mesh filename="package://luh_youbot_description/meshes/youbot_gripper/palm_convex.dae" />
-                </geometry>
-            </collision>
-        </link>
-        <joint name="${name}_finger_joint_l" type="prismatic">
-            <origin xyz="0.004 0.007 0.0115" rpy="0 0 ${M_PI}" />
-            <parent link="${name}_palm_link"/>
-            <child link="${name}_finger_link_l"/>
-            <axis xyz="0 -1 0" />
-            <dynamics damping="1.0" friction="1.0" />
-            <limit effort="1" velocity="0.1" lower="0" upper="${finger_joint}"/>
-            <safety_controller k_position="20" k_velocity="25" soft_lower_limit="${threshold}" soft_upper_limit="${finger_joint_soft}" />
-        </joint>
-        <link name="${name}_finger_link_l">
-            <inertial>
-                <origin xyz="0 0.00 0" rpy="0 0 0" />
-                <mass value="0.01"/>
-                <inertia ixx="0.00001" ixy="0" ixz="0" iyy="0.00001" iyz="0" izz="0.00001" />
-            </inertial>
-            <visual>
-                <origin xyz="0 0 0" rpy="0 ${-M_PI/2} 0" /> <!---->
-                <geometry>
-                    <mesh filename="package://luh_youbot_description/meshes/youbot_gripper/finger.dae" />
-                </geometry>
-            </visual>
-            <collision>
-                <origin xyz="0 0 0" rpy="0 ${-M_PI/2} 0" />
-                <geometry>
-                    <mesh filename="package://luh_youbot_description/meshes/youbot_gripper/finger_convex.dae" />
-                </geometry>
-            </collision>
-        </link>
+	<xacro:include filename="$(find luh_youbot_description)/urdf/youbot_gripper/limits.urdf.xacro" />
+	<xacro:include filename="$(find luh_youbot_description)/urdf/youbot_gripper/gripper.gazebo.xacro" />
+	<xacro:macro name="youbot_gripper" params="parent name namespace *origin">
+		<!-- joint between arm_7_link and sdh_palm_link -->
+		<joint name="${name}_palm_joint" type="fixed" >
+			<insert_block name="origin" />
+			<parent link="${parent}" />
+			<child link="${name}_palm_link" />
+		</joint>
+		<link name="${name}_palm_link">
+			<inertial>
+				<origin xyz="0 0 0" rpy="0 0 0"/>
+				<mass value="0.1"/>
+				<inertia ixx="0.01" ixy="0" ixz="0" iyy="0.01" iyz="0" izz="0.01" />
+			</inertial>
+			<visual>
+				<origin xyz="0 0 -0.0139" rpy="0 ${-M_PI/2} ${M_PI/2}"/>
+				<geometry>
+					<mesh filename="package://luh_youbot_description/meshes/youbot_gripper/palm.dae" />
+				</geometry>
+			</visual>
+			<collision>
+				<origin xyz="0.003 0 0.01" rpy="0 0 0" />
+				<geometry>
+					<!-- <mesh filename="package://luh_youbot_description/meshes/youbot_gripper/palm_convex.dae" /> -->
+					<box size="0.0001 0.0001 0.0001" />
+				</geometry>
+			</collision>
+		</link>
+		<joint name="${name}_finger_joint_l" type="prismatic">
+			<origin xyz="0.004 0.007 0.0115" rpy="0 0 ${M_PI}" />
+			<parent link="${name}_palm_link"/>
+			<child link="${name}_finger_link_l"/>
+			<axis xyz="0 -1 0" />
+			<dynamics damping="1.0" friction="1.0" />
+			<limit effort="1" velocity="0.1" lower="0" upper="${finger_joint}"/>
+                        <safety_controller k_position="20" k_velocity="25" soft_lower_limit="${threshold}" soft_upper_limit="${finger_joint_soft}" />
+		</joint>
+		<gazebo reference="gripper_finger_joint_l">
+    		<implicitSpringDamper>1</implicitSpringDamper>
+  		</gazebo>
+		<link name="${name}_finger_link_l">
+			<inertial>
+				<origin xyz="0 0.00 0" rpy="0 0 0" />
+				<mass value="0.01"/>
+				<inertia ixx="0.01" ixy="0" ixz="0" iyy="0.01" iyz="0" izz="0.01" />
+			</inertial>
+			<visual>
+				<origin xyz="0 0 0" rpy="0 ${-M_PI/2} 0" /> <!---->
+				<geometry>
+					<mesh filename="package://luh_youbot_description/meshes/youbot_gripper/finger.dae" />
+				</geometry>
+			</visual>
+			<collision>
+				<origin xyz="0 0 0" rpy="0 ${-M_PI/2} 0" />
+				<geometry>
+					<mesh filename="package://luh_youbot_description/meshes/youbot_gripper/finger_convex.dae" />
+				</geometry>
+			</collision>
+		</link>
+		<gazebo reference='gripper_finger_link_l'><maxVel>0.0</maxVel><fdir1>1.00000 1.00000 1.00000</fdir1><kp>1000000.0</kp><kd>1.0</kd><minDepth>0.001</minDepth><mu1>200.0</mu1>
+        <mu2>200.0</mu2></gazebo>
         <joint name="${name}_finger_joint_r" type="prismatic">
-            <origin xyz="0.004 -0.007 0.0115" rpy="0 0 0" />
-            <parent link="${name}_palm_link"/>
-            <child link="${name}_finger_link_r"/>
-            <axis xyz="0 -1 0" />
-            <dynamics damping="1.0" friction="1.0" />
-            <limit effort="1" velocity="0.1" lower="0" upper="${finger_joint}"/>
-            <safety_controller k_position="20" k_velocity="25" soft_lower_limit="${threshold}" soft_upper_limit="${finger_joint_soft}" />
-        </joint>
-        <link name="${name}_finger_link_r">
-            <inertial>
-                <origin xyz="0.000 -0.001 0" rpy="0 0 0" />
-                <mass value="0.01"/>
-                <inertia ixx="0.00001" ixy="0" ixz="0" iyy="0.0001" iyz="0" izz="0.00001" />
-            </inertial>
-            <visual>
-                <origin xyz="0 0 0" rpy="0 ${-M_PI/2} 0" /> <!-- -->
-                <geometry>
-                    <mesh filename="package://luh_youbot_description/meshes/youbot_gripper/finger.dae" />
-                </geometry>
-            </visual>
-            <collision>
-                <origin xyz="0 0 0" rpy="0 ${-M_PI/2} 0" />
-                <geometry>
-                    <mesh filename="package://luh_youbot_description/meshes/youbot_gripper/finger_convex.dae" />
-                </geometry>
-            </collision>
-        </link>
-        <!-- coordinate frame on the tip of the robot's gripper -->
-        <joint name="${name}_tip_joint" type="fixed">
-            <origin xyz="0.000 0 0.09" rpy="0.0 ${-M_PI / 2} 0.0" />
-            <parent link="${name}_palm_link" />
-            <child link="${name}_tip"/>
-        </joint>
-        <link name="${name}_tip">
-            <inertial>
-                <mass value="0.001" />
-                <origin xyz="0 0 0" />
-                <inertia ixx="0.000001" ixy="0.0" ixz="0.0" iyy="0.000001" iyz="0.0" izz="0.000001" />
-            </inertial>
-        </link>
+			<origin xyz="0.004 -0.007 0.0115" rpy="0 0 0" />
+			<parent link="${name}_palm_link"/>
+			<child link="${name}_finger_link_r"/>
+			<axis xyz="0 -1 0" />
+			<dynamics damping="1.0" friction="1.0" />
+			<limit effort="1" velocity="0.1" lower="0" upper="${finger_joint}"/>
+                        <safety_controller k_position="20" k_velocity="25" soft_lower_limit="${threshold}" soft_upper_limit="${finger_joint_soft}" />
+		</joint>
+		<gazebo reference="gripper_finger_joint_r">
+    		<implicitSpringDamper>1</implicitSpringDamper>
+  		</gazebo>
+		<link name="${name}_finger_link_r">
+			<inertial>
+				<origin xyz="0.000 -0.001 0" rpy="0 0 0" />
+				<mass value="0.01"/>
+				<inertia ixx="0.01" ixy="0" ixz="0" iyy="0.01" iyz="0" izz="0.01" />
+			</inertial>
+			<visual>
+				<origin xyz="0 0 0" rpy="0 ${-M_PI/2} 0" /> <!-- -->
+				<geometry>
+					<mesh filename="package://luh_youbot_description/meshes/youbot_gripper/finger.dae" />
+				</geometry>
+			</visual>
+			<collision>
+				<origin xyz="0 0 0" rpy="0 ${-M_PI/2} 0" />
+				<geometry>
+					<mesh filename="package://luh_youbot_description/meshes/youbot_gripper/finger_convex.dae" />
+				</geometry>
+			</collision>
+		</link>
+		  <gazebo reference='gripper_finger_link_r'><maxVel>0.0</maxVel><fdir1>1.00000 1.00000 1.00000</fdir1><kp>1000000.0</kp><kd>1.0</kd><minDepth>0.001</minDepth><mu1>200.0</mu1>
+        <mu2>200.0</mu2></gazebo>
+		<!-- coordinate frame on the tip of the robot's gripper -->
+		<joint name="${name}_tip_joint" type="fixed">
+			<origin xyz="0.000 0 0.09" rpy="0.0 ${-M_PI / 2} 0.0" />
+			<parent link="${name}_palm_link" />
+			<child link="${name}_tip"/>
+		</joint>
+		<link name="${name}_tip">
+			<inertial>
+				<mass value="0.001" />
+				<origin xyz="0 0 0" />
+				<inertia ixx="0.001" ixy="0.0" ixz="0.0" iyy="0.001" iyz="0.0" izz="0.001" />
+			</inertial>
+		</link>
                 <xacro:youbot_gripper_controller namespace="${namespace}"/>
-    </xacro:macro>
+	</xacro:macro>
 </robot>

Commit message: worked for kai's demo

File: luh_youbot_description/robots/youbot.urdf.xacro (robot description, xacro)
@@ -17,5 +17,6 @@
   <xacro:youbot_base name="base" namespace="youbot_0"/>
   <xacro:youbot_plate name="plate" parent="base_link">
-    <origin xyz="-0.039 0 0.064" rpy="0 0 0" />
+    <origin rpy="0 0 0" xyz="-0.159 0 0.046"/>
+    <!-- <origin xyz="-0.039 0 0.064" rpy="0 0 0" /> -->
   </xacro:youbot_plate>
   <xacro:youbot_arm name="arm" parent="base_link" namespace="youbot_0">
