Commit message: removed unnecessary mode for BaseController; added MultiBaseController, untested; updated forklift

File: youbot_forklift/youbot_forklift_description/robots/youbot_with_forklift.urdf.xacro (robot description, xacro)
@@ -1,12 +1,9 @@
 <?xml version="1.0"?>
-<robot xmlns:sensor="http://playerstage.sourceforge.net/gazebo/xmlschema/#sensor"
-       xmlns:controller="http://playerstage.sourceforge.net/gazebo/xmlschema/#controller"
-       xmlns:interface="http://playerstage.sourceforge.net/gazebo/xmlschema/#interface"
-       xmlns:xacro="http://ros.org/wiki/xacro"
-       name="youbot" >
+<robot name="youbot" xmlns:xacro="http://www.ros.org/wiki/xacro">
   <xacro:include filename="$(find luh_youbot_description)/urdf/common.xacro" />
 	<xacro:include filename="$(find youbot_forklift_description)/controller/ros_controller.urdf.xacro" />
 	<xacro:include filename="$(find youbot_forklift_description)/urdf/youbot_forklift/forklift.urdf.xacro"/>
 	<xacro:include filename="$(find luh_youbot_description)/urdf/youbot_base/base.urdf.xacro" />
+  <xacro:include filename="$(find luh_youbot_description)/urdf/youbot_plate/plate.urdf.xacro" />
 	<!-- <xacro:include filename="$(find luh_youbot_description)/urdf/materials.urdf.xacro" /> -->
  <xacro:youbot_base name="base"  namespace="youbot_2"/>
@@ -14,3 +11,6 @@
     <origin xyz="0 0 -0.075" rpy="0 0 0"/>
 	</xacro:youbot_forklift>
+  <xacro:youbot_plate name="plate" parent="base_link">
+    <origin xyz="-0.039 0 0.064" rpy="0 0 0" />
+  </xacro:youbot_plate>
 </robot>
